Commit message: refactor(models): update leader arm v2 model and fix x500 propellers

File: neutele/station/flying_hand/urdf/leader/leader.urdf (robot description, URDF)
Before this commit: robot flying_hand_leader, 6 links, 5 joints
Links:
- link base_link: mass 0.13025 -> 0.1139
- link link_1: mass 0.08581 -> 0.1468
- link link_2: mass 0.11524 -> 0.1467
- link link_3: mass 0.0848 -> 0.0618
- link link_4: mass 0.0542 -> 0.0518
Joints:
- joint joint_1: limit lower=-2.8973 upper=2.8973 effort=3.43 velocity=4.72 -> lower=-2.6485 upper=2.6485 effort=4.9008 velocity=8.95; origin xyz=0 0 0.0528 rpy=0 0 0 -> xyz=0.004 -0.0005 0.04811 rpy=1.5708 0 3.1416
- joint joint_2: limit lower=-1.7628 upper=1.7628 effort=4.903 velocity=8.95 -> lower=0 upper=3.4907 effort=3.4305 velocity=4.72; origin xyz=0 0 0.0486100000000001 rpy=1.5707963267949 0 3.14159265358979 -> xyz=-0.04098 0.2314 -0.0005 rpy=0 0 0
- joint joint_3: limit lower=0 upper=1.7628 effort=3.43 velocity=4.72 -> lower=-2.6485 upper=2.6485 effort=3.4305 velocity=4.72; origin xyz=-0.0381400000000001 0.1640000018731 -0.000200000000001629 rpy=0 0 0 -> xyz=0.04098 0.24861 -0.0005 rpy=0 0 0
- joint joint_4: axis 0 0 -1 -> 0 0 1; limit lower=-2.8973 upper=2.8973 effort=1.39 velocity=10.47 -> lower=-3.1416 upper=3.1416 effort=1.3918 velocity=10.47; origin xyz=0.03582 0.1935 -0.00077 rpy=1.5708 0 -3.1416 -> xyz=0 0.0639 0 rpy=1.5708 -1.5708 0
- joint joint_5: axis 0 0 -1 -> 0 0 1; limit lower=-2.8973 upper=2.8973 effort=1.471 velocity=7.12 -> lower=-1.7628 upper=0 effort=1.3918 velocity=10.47; origin xyz=0 0.02485 0.03 rpy=1.5708 0 0 -> xyz=0.01315 0.0005 -0.047756 rpy=-1.5708 0 -1.5708

File: neutele/station/flying_hand/urdf/x500_arm/x500_arm.urdf (robot description, URDF)
Before this commit: robot x500_arm, 10 links, 9 joints
Links:
- added link world
- link link_1: mass 0.07754703 -> 0.1468
- link link_2: mass 0.06972203 -> 0.1467
- link link_3: mass 0.04826195 -> 0.0618
- link link_4: mass 0.02233811 -> 0.022338
Joints:
- added joint floating_base_joint: type floating, parent world, child base_link, origin xyz=0 0 0 rpy=0 0 0
- joint joint_2: origin xyz=0.04048 -0.2314 -0.0005 rpy=0 0 0 -> xyz=0.04098 -0.2314 -0.0005 rpy=0 0 0
- joint joint_3: origin xyz=-0.0404 -0.24861 -0.0005 rpy=0 0 0 -> xyz=-0.04098 -0.24861 -0.0005 rpy=0 0 0
- joint joint_4: origin xyz=0 -0.0629 0 rpy=1.5708 -1.5708 0 -> xyz=0 -0.0639 0 rpy=1.5708 -1.5708 0
- joint joint_5: origin xyz=0 -0.0044 0.02243 rpy=-1.5708 0 -1.5708 -> xyz=-0.0044 0 0.02243 rpy=-1.5708 0 0
- joint rotor_joint_1: origin xyz=0.17688 -0.17688 0.056 rpy=0 0 0 -> xyz=0.17688 -0.17688 0.066 rpy=0 0 0
- joint rotor_joint_2: origin xyz=0.17688 0.17688 0.056 rpy=0 0 0 -> xyz=0.17688 0.17688 0.066 rpy=0 0 0
- joint rotor_joint_3: origin xyz=-0.17688 0.17688 0.056 rpy=0 0 0 -> xyz=-0.17688 0.17688 0.066 rpy=0 0 0
- joint rotor_joint_4: origin xyz=-0.17688 -0.17688 0.056 rpy=0 0 0 -> xyz=-0.17688 -0.17688 0.066 rpy=0 0 0
