Commit message: fix(core): align initial pose with home pose

File: acetele/station/follower/description/follower.urdf (robot description, URDF)
Before this commit: robot follower, 7 links, 6 joints
Links:
- link base_link: geometry collision mesh filename=meshes/base_link.STL; visual mesh filename=meshes/base_link.STL
- link link_1: geometry collision mesh filename=meshes/link_1.STL; visual mesh filename=meshes/link_1.STL
- link link_2: geometry collision mesh filename=meshes/link_2.STL; visual mesh filename=meshes/link_2.STL
- link link_3: geometry collision mesh filename=meshes/link_3.STL; visual mesh filename=meshes/link_3.STL
- link link_4: geometry collision mesh filename=meshes/link_4.STL; visual mesh filename=meshes/link_4.STL
- link link_5_left: geometry collision mesh filename=meshes/link_5_left.STL; visual mesh filename=meshes/link_5_left.STL
- link link_5_right: geometry collision mesh filename=meshes/link_5_right.STL; visual mesh filename=meshes/link_5_right.STL
