Commit message: refactor(urdf): replace follower model with x500 arm

File: acetele/robot/ace_follower/description/ace_follower.urdf (robot description, URDF)
Before this commit: robot ace_follower, 6 links, 5 joints
Links:
- link base_link: mass 1.7698 -> None; geometry 
- link link_1: mass 0.05836 -> 0.15156
- link link_2: mass 0.05486 -> 0.14766
- link link_3: mass 0.04246 -> 0.0636
- link link_4: mass 0.0544 -> 0.11656
- link link_5: mass 0.0045 -> 0.0035
Joints:
- joint joint_1: limit lower=-2.6485 upper=2.6485 effort=1.3918 velocity=10.47 -> lower=-2.6485 upper=2.6485 effort=5.24 velocity=6.28; origin xyz=-0.00015 0.00015 0.4085 rpy=1.5708 0 0 -> xyz=0 0.0002 -0.1453 rpy=-1.5708 0 3.1416
- joint joint_2: limit lower=0 upper=3.4907 effort=1.3918 velocity=10.47 -> lower=0 upper=3.4907 effort=3.92 velocity=7.85; origin xyz=0.02064 -0.1157 -0.00015 rpy=0 0 0 -> xyz=-0.04098 0.2314 -0.0005 rpy=0 0 3.1416
- joint joint_3: limit lower=-2.6485 upper=2.6485 effort=1.3918 velocity=10.47 -> lower=-2.6485 upper=2.6485 effort=2.75 velocity=4.71; origin xyz=-0.02034 -0.12431 -0.00015 rpy=0 0 0 -> xyz=-0.04098 -0.26861 0 rpy=0 0 0
- joint joint_4: limit lower=-3.1416 upper=3.1416 effort=1.3918 velocity=10.47 -> lower=-3.1416 upper=3.1416 effort=1.11 velocity=10.47; origin xyz=0.00015 -0.044 -0.00015 rpy=-1.5708 0 3.1416 -> xyz=0 -0.05189 0 rpy=1.5708 1.5708 0
- joint joint_5: limit lower=-3.1416 upper=0 effort=1.3918 velocity=10.47 -> lower=-1.723 upper=0 effort=1.11 velocity=10.47; origin xyz=0.0005 0.02005 0.0305 rpy=-1.5708 0 0 -> xyz=0 0 0.037 rpy=0 0 0
